File: NoteDetector/NoteDetector.kicad_sch (KiCad schematic)
At the start: 49 parts, among them J1 Conn_01x01, J2 Conn_01x01, J3 Conn_01x01, J4 Conn_01x01, J5 Conn_01x01, J6 Conn_01x01, J7 Conn_01x01, Q1 Q_NMOS_DGS, Q2 Q_NMOS_DGS, Q3 Q_NMOS_DGS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

Commit message: Changelog: combined midscale references; added reverse voltage protection; moved ~MCLR programming pad to board perimeter; increased min drill/pad size
Parts:
- removed C3, C4: 1n, Capacitor_SMD:C_0603_1608Metric, symbol Device:C
- removed R6: 1k, Resistor_SMD:R_0603_1608Metric, symbol Device:R
- removed R7, R8: 10M, Resistor_SMD:R_0603_1608Metric, symbol Device:R
- added Q5: Q_NMOS_DGS, Package_TO_SOT_SMD:SOT-23, symbol Device:Q_NMOS_GSD
- C5: value C_in -> 10n; Part Number (none) -> 0603B103J500CT; Part Number Alt 1 CL10B104JB8NNNC -> (none); Val1 10n -> (none); Val2 1.5n -> (none)
- C7, C8: value C_fb -> 10p; Part Number (none) -> 0603N100J500CT; Part Number Alt 1 06035A220JAT2A -> (none); Val1 22p -> (none); Val2 10p -> (none)
Connections:
- net Midscale2 is gone; now on net Midscale: C1.1, C2.2, R15.2, R4.1, R5.2
- net +BATT: now also Q5.1 (G)
- net GND: now also Q5.2 (S); no longer BT1.2 (-)
- net Midscale1 renamed Midscale
- new net PGnd: BT1.2 (-), Q5.3 (D)
Other:
- note added: "Reverse input protection"
